File: mk-ii-chokia/hardware/motherboard.brd (EAGLE design)
At the start: 256.2 x 198.1 mm, 24 parts, among them SW1 CHERRY_MX, SW10 CHERRY_MX, SW11 CHERRY_MX, SW12 CHERRY_MX, SW13 CHERRY_MX, SW14 CHERRY_MX, SW2 CHERRY_MX, SW3 CHERRY_MX, SW4 CHERRY_MX, SW5 CHERRY_MX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

Commit message: PCB trackin'
Parts:
- removed R1: 10k, rcl:0204/5
- added JP2: (no value), pinhead:1X02/90
- added R2: 10k, resistor-power:AC01
- added SW15: CHERRY_MX, Cherry_MX_v7.0:MX1A-XXNN
- moved SW12 349.0 mm to (72.4, 27.9), flipped to the bottom
- moved SW11 327.4 mm to (53.3, 27.9), flipped to the bottom
- moved SW14 318.5 mm to (38.1, 8.89), flipped to the bottom
- moved SW10 306.4 mm to (34.3, 27.9), flipped to the bottom
- moved SW13 292.4 mm to (15.2, 8.89), flipped to the bottom
- moved SW6 281.5 mm to (72.4, 47.0), flipped to the bottom
- moved SW9 271.1 mm to (15.2, 27.9), flipped to the bottom
- moved SW8 257.8 mm to (15.2, 47.0), flipped to the bottom
- moved SW5 246.6 mm to (53.3, 47.0), flipped to the bottom
- moved SW7 246.3 mm to (15.2, 66.0), flipped to the bottom
- moved T2 222.2 mm to (80.0, 104.1)
- moved U$3 150.1 mm to (5.08, 142.2), turned to 270 degrees
- moved R3 108.7 mm to (14.0, 99.1), turned to 270 degrees
- moved U$4 96.6 mm to (73.7, 135.9)
- moved U$5 93.2 mm to (73.7, 91.4)
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Connections:
- new net N$28: SW13.1, U$2.P$3
- new net N$32: JP2.1, U$3.B+
- new net N$33: JP2.2, U$3.B-
- net GND: now also SW15.2
- net N$13: now also R2.2; no longer R1.2
- net N$18: now also R2.1; no longer R1.1
- net N$29: now also SW15.1, U$2.P$2; no longer SW13.1, U$2.P$3
Routing:
- net N$29: track 0.00 -> 252.9 mm
- net N$31: track 0.00 -> 227.9 mm
- net N$30: track 0.00 -> 202.7 mm
- net N$28: track 0.00 -> 183.2 mm
- net N$27: track 0.00 -> 177.5 mm
- net N$22: track 0.00 -> 156.4 mm
- net N$26: track 0.00 -> 150.9 mm
- net N$21: track 0.00 -> 130.5 mm
- net N$19: track 0.00 -> 124.3 mm
- net N$25: track 0.00 -> 123.2 mm
- net N$20: track 0.00 -> 104.5 mm
- net N$23: track 0.00 -> 99.8 mm
- net N$17: track 0.00 -> 98.4 mm
- net N$15: track 0.00 -> 72.5 mm
- net N$24: track 0.00 -> 68.4 mm
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- added copper zone on layer 16, net GND
Other:
- board size 256.2 x 198.1 mm -> 100 x 165.1 mm

Commit message: Ready 2 etch dot com?
Parts:
- moved U$3 72.7 mm to (77.5, 135.9), turned to 180 degrees
- moved JP1 64.9 mm to (57.1, 128.3)
- moved JP2 62.3 mm to (57.1, 138.4)
- moved U$4 47.5 mm to (26.2, 135.9)
- moved U$2 37.1 mm to (17.8, 105.4), turned to 90 degrees
- moved R7 34.7 mm to (26.7, 124.5), flipped to the top, turned to 0 degrees
- moved R3 25.0 mm to (26.7, 120.7), turned to 180 degrees
- moved R2 15.3 mm to (57.1, 118.1)
- moved T2 13.1 mm to (86.4, 115.6)
- moved U$1 2.54 mm to (43.2, 111.8)
- moved U$5 1.27 mm to (73.7, 92.7)
Routing:
- net N$29: track 252.9 -> 188.1 mm
- net +5V: track 26.5 -> 88.5 mm
- net N$28: track 183.2 -> 121.3 mm
- net N$31: track 227.9 -> 168.8 mm
- net N$24: track 68.4 -> 11.4 mm
- net N$30: track 202.7 -> 146.4 mm
- net N$27: track 177.5 -> 124.1 mm
- net N$16: track 2.69 -> 56.1 mm
- net N$26: track 150.9 -> 101.8 mm
- net N$25: track 123.2 -> 87.1 mm
- net N$4: track 0.00 -> 34.3 mm
- net N$23: track 99.8 -> 67.3 mm
- net N$5: track 0.00 -> 31.2 mm
- net N$11: track 52.6 -> 83.2 mm
- net N$6: track 0.00 -> 28.2 mm
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Other:
- board size 100 x 165.1 mm -> 93 x 148.6 mm

Commit message: dump
Parts:
- added S1: (no value), switch-omron:B3F-10XX
- moved U$5 12.7 mm to (73.7, 105.4)
- moved SW15 3.54 mm to (65.0, 8.89)
- moved SW14 2.95 mm to (41.1, 8.89)
Connections:
- new net N$34: S1.3, U$2.P$18
- net +5V: now also S1.1; no longer U$2.P$18
Routing:
- net N$29: track 188.1 -> 172.5 mm
- net +5V: track 88.5 -> 103.0 mm
- net N$16: track 56.1 -> 43.4 mm
- net N$34: track 0.00 -> 11.8 mm
- net N$22: track 141.9 -> 131.4 mm
- net N$28: track 121.3 -> 112.9 mm
- net N$21: track 118.5 -> 110.3 mm
- net N$4: track 34.3 -> 41.2 mm
- net N$20: track 95.1 -> 89.3 mm
- net N$19: track 117.4 -> 111.8 mm
- net N$5: track 31.2 -> 36.0 mm
- net +3V3: track 83.4 -> 88.2 mm
- net N$31: track 168.8 -> 164.9 mm
- net N$25: track 87.1 -> 90.8 mm
- net N$6: track 28.2 -> 31.9 mm
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