File: mk-ii-chokia/hardware/motherboard.sch (EAGLE design)
At the start: 10 parts, among them T2 BC337

Commit message: Chokia sends. Pager receives. Not vice-versa...
Connections:
- removed net N$31: T2.E, U$1.A_LED_+5V
- new net N$14: T2.C, U$1.K_LED_0V
- new net N$17: U$2.PA10
- net +5V: now also U$1.A_LED_+5V
- net GND: now also T2.E; no longer U$1.K_LED_0V
- net N$15: now also U$2.PA9; no longer T2.C
- net N$18: now also U$2.PA0; no longer U$2.PC15
Other:
- moved on the sheet: R1, T2
Changed lines of the file:
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@@
 <attribute name="VALUE" x="111.76" y="91.44" size="1.778" layer="96"/>
 </instance>
-<instance part="GND11" gate="1" x="114.3" y="40.64" smashed="yes">
-<attribute name="VALUE" x="111.76" y="38.1" size="1.778" layer="96"/>
+<instance part="GND11" gate="1" x="104.14" y="25.4" smashed="yes">
+<attribute name="VALUE" x="101.6" y="22.86" size="1.778" layer="96"/>
 </instance>
 <instance part="P+3" gate="1" x="109.22" y="93.98" smashed="yes">
 <attribute name="VALUE" x="106.68" y="88.9" size="1.778" layer="96" rot="R90"/>
 </instance>
-<instance part="T2" gate="G$1" x="104.14" y="43.18" smashed="yes">
-<attribute name="NAME" x="101.6" y="50.8" size="1.778" layer="95"/>
-<attribute name="VALUE" x="101.6" y="48.26" size="1.778" layer="96"/>
-</instance>
-<instance part="R1" gate="G$1" x="96.52" y="43.18" smashed="yes">
-<attribute name="NAME" x="92.71" y="44.6786" size="1.778" layer="95"/>
-<attribute name="VALUE" x="92.71" y="39.878" size="1.778" layer="96"/>
+<instance part="T2" gate="G$1" x="101.6" y="35.56" smashed="yes">
+<attribute name="NAME" x="99.06" y="43.18" size="1.778" layer="95"/>
+<attribute name="VALUE" x="99.06" y="40.64" size="1.778" layer="96"/>
+</instance>
+<instance part="R1" gate="G$1" x="91.44" y="35.56" smashed="yes">
+<attribute name="NAME" x="87.63" y="37.0586" size="1.778" layer="95"/>
+<attribute name="VALUE" x="87.63" y="32.258" size="1.778" layer="96"/>
 </instance>
 <instance part="P+4" gate="1" x="106.68" y="50.8" smashed="yes">
@@
 </segment>
 <segment>
+<pinref part="T2" gate="G$1" pin="E"/>
 <pinref part="GND11" gate="1" pin="GND"/>
-<pinref part="U$1" gate="G$1" pin="K_LED_0V"/>
-<wire x1="114.3" y1="43.18" x2="119.38" y2="43.18" width="0.1524" layer="91"/>
-<wire x1="119.38" y1="43.18" x2="119.38" y2="45.72" width="0.1524" layer="91"/>
+<wire x1="104.14" y1="30.48" x2="104.14" y2="27.94" width="0.1524" layer="91"/>
 </segment>
 </net>
@@
 <pinref part="U$1" gate="G$1" pin="VDD_+5V"/>
 <wire x1="109.22" y1="91.44" x2="119.38" y2="91.44" width="0.1524" layer="91"/>
+</segment>
+<segment>
+<pinref part="U$1" gate="G$1" pin="A_LED_+5V"/>
+<wire x1="106.68" y1="48.26" x2="119.38" y2="48.26" width="0.1524" layer="91"/>
+<pinref part="P+4" gate="1" pin="+5V"/>
 </segment>
 </net>
@@
 <pinref part="T2" gate="G$1" pin="B"/>
 <pinref part="R1" gate="G$1" pin="2"/>
+<wire x1="96.52" y1="35.56" x2="99.06" y2="35.56" width="0.1524" layer="91"/>
+</segment>
+</net>
+<net name="N$18" class="0">
+<segment>
+<pinref part="U$2" gate="G$1" pin="PA0"/>
+<wire x1="83.82" y1="55.88" x2="86.36" y2="55.88" width="0.1524" layer="91"/>
+<pinref part="R1" gate="G$1" pin="1"/>
+<wire x1="86.36" y1="35.56" x2="86.36" y2="55.88" width="0.1524" layer="91"/>
+</segment>
+</net>
+<net name="N$14" class="0">
+<segment>
+<pinref part="U$1" gate="G$1" pin="K_LED_0V"/>
+<pinref part="T2" gate="G$1" pin="C"/>
+<wire x1="119.38" y1="45.72" x2="104.14" y2="45.72" width="0.1524" layer="91"/>
+<wire x1="104.14" y1="45.72" x2="104.14" y2="40.64" width="0.1524" layer="91"/>
 </segment>
 </net>
 <net name="N$15" class="0">
 <segment>
-<pinref part="T2" gate="G$1" pin="C"/>
-<pinref part="P+4" gate="1" pin="+5V"/>
-</segment>
-</net>
-<net name="N$18" class="0">
-<segment>
-<pinref part="U$2" gate="G$1" pin="PC15"/>
-<wire x1="83.82" y1="53.34" x2="91.44" y2="53.34" width="0.1524" layer="91"/>
-<pinref part="R1" gate="G$1" pin="1"/>
-<wire x1="91.44" y1="53.34" x2="91.44" y2="43.18" width="0.1524" layer="91"/>
-</segment>
-</net>
-<net name="N$31" class="0">
-<segment>
-<pinref part="T2" gate="G$1" pin="E"/>
-<wire x1="106.68" y1="38.1" x2="109.22" y2="38.1" width="0.1524" layer="91"/>
-<wire x1="109.22" y1="38.1" x2="109.22" y2="48.26" width="0.1524" layer="91"/>
-<pinref part="U$1" gate="G$1" pin="A_LED_+5V"/>
-<wire x1="109.22" y1="48.26" x2="119.38" y2="48.26" width="0.1524" layer="91"/>
-</segment>
-</net>
+<pinref part="U$2" gate="G$1" pin="PA9"/>
+<wire x1="43.18" y1="81.28" x2="40.64" y2="81.28" width="0.1524" layer="91"/>
+</segment>
+</net>
+<net name="N$17" class="0">
+<segment>
+<pinref part="U$2" gate="G$1" pin="PA10"/>
+<wire x1="43.18" y1="78.74" x2="40.64" y2="78.74" width="0.1524" layer="91"/>
+</segment>
+</net>

Commit message: Eagle grief and keycaps
Parts:
- added SW1, SW10, SW11, SW12, SW13, SW14, SW2, SW3, SW4, SW5, SW6, SW7, SW8, SW9: CHERRY_MX, Cherry_MX_v7.0:CHERRY_MX
Connections:
- new net N$19: SW3.1, U$2.PB7
- new net N$20: SW4.1, U$2.PB6
- new net N$21: SW5.1, U$2.PB5
- new net N$22: SW6.1, U$2.PB4
- new net N$23: SW7.1, U$2.PB3
- new net N$25: SW8.1, U$2.PA15
- new net N$26: SW9.1, U$2.PA10
- new net N$27: SW10.1, U$2.PA9
- new net N$29: SW13.1, SW14.1, U$2.PB14
- new net N$30: SW11.1, U$2.PA8
- new net N$31: SW12.1, U$2.PB15
- net GND: now also SW1.2, SW10.2, SW11.2, SW12.2, SW13.2, SW14.2, SW2.2, SW3.2, SW4.2, SW5.2, SW6.2, SW7.2, SW8.2, SW9.2
- net N$15: now also SW1.1, U$2.PB9; no longer U$2.PA9
- net N$17: now also SW2.1, U$2.PB8; no longer U$2.PA10
- net N$24: now also U$2.PB1; no longer U$2.PA15
- net N$3: now also U$2.PB11, U$4.RESET; no longer U$4.SCK
- net N$4: now also U$2.PB0, U$4.NSS; no longer U$4.MISO
- net N$5: now also U$2.PA7
- net N$6: now also U$2.PA6, U$4.MISO; no longer U$4.NSS
- net N$7: now also U$2.PA5, U$4.SCK; no longer U$4.DIO0
- net N$8: now also U$2.PB10, U$4.DIO0; no longer U$4.RESET
Other:
- moved on the sheet: U$4

Commit message: PCB trackin'
Parts:
- removed R1: 10k, rcl:R-EU_0204/5
- added JP2: (no value), pinhead:PINHD-1X2/90
- added R2: 10k, resistor-power:RAC01
- added SW15: CHERRY_MX, Cherry_MX_v7.0:CHERRY_MX
Connections:
- new net N$28: SW13.1, U$2.PB14
- new net N$32: JP2.1, U$3.B+
- new net N$33: JP2.2, U$3.B-
- net GND: now also SW15.2
- net N$13: now also R2.2; no longer R1.2
- net N$18: now also R2.1; no longer R1.1
- net N$29: now also SW15.1, U$2.PB13; no longer SW13.1, U$2.PB14

Commit message: dump
Parts:
- added S1: (no value), switch-omron:10-XX
Connections:
- new net N$34: S1.P, U$2.5V
- net +5V: now also S1.S; no longer U$2.5V
Changed lines of the file:
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@@
 <part name="SW14" library="Cherry_MX_v7.0" deviceset="CHERRY_MX" device=""/>
 <part name="SW15" library="Cherry_MX_v7.0" deviceset="CHERRY_MX" device=""/>
+<part name="S1" library="switch-omron" library_urn="urn:adsk.eagle:library:377" deviceset="10-XX" device="" package3d_urn="urn:adsk.eagle:package:27496/1"/>
 </parts>
 <sheets>
@@
 <attribute name="VALUE" x="10.16" y="7.62" size="1.778" layer="96" rot="R90"/>
 </instance>
-<instance part="P+2" gate="1" x="25.4" y="50.8" smashed="yes">
-<attribute name="VALUE" x="25.4" y="43.18" size="1.778" layer="96" rot="R90"/>
+<instance part="P+2" gate="1" x="22.86" y="50.8" smashed="yes">
+<attribute name="VALUE" x="22.86" y="43.18" size="1.778" layer="96" rot="R90"/>
 </instance>
 <instance part="U$4" gate="P$1" x="60.96" y="147.32" smashed="yes" rot="R180">
@@
 <instance part="SW14" gate="G$1" x="5.08" y="119.38" smashed="yes" rot="R270"/>
 <instance part="SW15" gate="G$1" x="5.08" y="114.3" smashed="yes" rot="R270"/>
+<instance part="S1" gate="1" x="22.86" y="43.18" smashed="yes">
+<attribute name="NAME" x="16.51" y="40.64" size="1.778" layer="95" rot="R90"/>
+<attribute name="VALUE" x="19.05" y="46.355" size="1.778" layer="96" rot="R90"/>
+</instance>
 </instances>
 <busses>
@@
 <segment>
 <pinref part="P+2" gate="1" pin="+5V"/>
-<pinref part="U$2" gate="G$1" pin="5V"/>
-<wire x1="43.18" y1="50.8" x2="30.48" y2="50.8" width="0.1524" layer="91"/>
-<wire x1="30.48" y1="50.8" x2="30.48" y2="48.26" width="0.1524" layer="91"/>
-<wire x1="30.48" y1="48.26" x2="25.4" y2="48.26" width="0.1524" layer="91"/>
+<pinref part="S1" gate="1" pin="S"/>
 </segment>
 <segment>
@@
 </segment>
 </net>
+<net name="N$34" class="0">
+<segment>
+<pinref part="U$2" gate="G$1" pin="5V"/>
+<wire x1="43.18" y1="50.8" x2="30.48" y2="50.8" width="0.1524" layer="91"/>
+<wire x1="30.48" y1="50.8" x2="30.48" y2="35.56" width="0.1524" layer="91"/>
+<pinref part="S1" gate="1" pin="P"/>
+<wire x1="22.86" y1="38.1" x2="22.86" y2="35.56" width="0.1524" layer="91"/>
+<wire x1="22.86" y1="35.56" x2="30.48" y2="35.56" width="0.1524" layer="91"/>
+</segment>
+</net>
